File: Electronics/idp.brd (EAGLE design)
At the start: 100 x 80 mm, 6 parts, among them J1 22-05-7048-04, M1 IDP_PROTOBOARD

Commit message: Updated eagle schematics
Parts:
- added IC1: LM311N, IDP_library:DIL08
- added LED2, LED3, LED4, LED5: LED_23MM, IDP_library:LED3MM
- added R3, R4, R5, R6: R-EU_0207/5V, IDP_library:0207/5V
- added U$2: HALL-SS495A, IDP_library:TO92/
Connections:
- new net N$1: LED2.A, R3.2
- new net N$2: LED3.A, R4.2
- new net N$4: LED4.A, R5.2
- new net N$5: LED5.A, R6.2
- new net N$8: IC1.2, U$2.1
- new net V+: IC1.8
- new net V-: IC1.4
- net +5V: now also U$2.3
- net D0: now also R6.1
- net D1: now also R5.1
- net D2: now also R4.1
- net D3: now also R3.1
- net GND: now also LED2.K, LED3.K, LED4.K, LED5.K, U$2.2
Changed lines of the file:
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@@
 <attribute name="VALUE" x="-11.8379" y="-115.4699" size="0.8128" layer="27" ratio="10" rot="R270"/>
+</element>
+<element name="R3" library="IDP_library" package="0207/5V" package3d_urn="urn:adsk.eagle:package:23502/1" value="R-EU_0207/5V" x="-19.05" y="-130.81" smashed="yes">
+<attribute name="NAME" x="-20.193" y="-129.921" size="1.27" layer="25" ratio="10"/>
+<attribute name="POPULARITY" value="4" x="-19.05" y="-130.81" size="1.778" layer="27" display="off"/>
+<attribute name="SPICEPREFIX" value="R" x="-19.05" y="-130.81" size="1.778" layer="27" display="off"/>
+<attribute name="VALUE" x="-20.193" y="-132.969" size="1.27" layer="27" ratio="10"/>
+</element>
+<element name="R4" library="IDP_library" package="0207/5V" package3d_urn="urn:adsk.eagle:package:23502/1" value="R-EU_0207/5V" x="-19.05" y="-137.16" smashed="yes">
+<attribute name="NAME" x="-20.193" y="-136.271" size="1.27" layer="25" ratio="10"/>
+<attribute name="POPULARITY" value="4" x="-19.05" y="-137.16" size="1.778" layer="27" display="off"/>
+<attribute name="SPICEPREFIX" value="R" x="-19.05" y="-137.16" size="1.778" layer="27" display="off"/>
+<attribute name="VALUE" x="-20.193" y="-139.319" size="1.27" layer="27" ratio="10"/>
+</element>
+<element name="R5" library="IDP_library" package="0207/5V" package3d_urn="urn:adsk.eagle:package:23502/1" value="R-EU_0207/5V" x="-19.05" y="-143.51" smashed="yes">
+<attribute name="NAME" x="-20.193" y="-142.621" size="1.27" layer="25" ratio="10"/>
+<attribute name="POPULARITY" value="4" x="-19.05" y="-143.51" size="1.778" layer="27" display="off"/>
+<attribute name="SPICEPREFIX" value="R" x="-19.05" y="-143.51" size="1.778" layer="27" display="off"/>
+<attribute name="VALUE" x="-20.193" y="-145.669" size="1.27" layer="27" ratio="10"/>
+</element>
+<element name="R6" library="IDP_library" package="0207/5V" package3d_urn="urn:adsk.eagle:package:23502/1" value="R-EU_0207/5V" x="-19.05" y="-149.86" smashed="yes">
+<attribute name="NAME" x="-20.193" y="-148.971" size="1.27" layer="25" ratio="10"/>
+<attribute name="POPULARITY" value="4" x="-19.05" y="-149.86" size="1.778" layer="27" display="off"/>
+<attribute name="SPICEPREFIX" value="R" x="-19.05" y="-149.86" size="1.778" layer="27" display="off"/>
+<attribute name="VALUE" x="-20.193" y="-152.019" size="1.27" layer="27" ratio="10"/>
+</element>
+<element name="LED2" library="IDP_library" package="LED3MM" package3d_urn="urn:adsk.eagle:package:15797/1" value="LED_23MM" x="-20.32" y="-154.94" smashed="yes">
+<attribute name="NAME" x="-18.415" y="-154.559" size="1.27" layer="25" ratio="10"/>
+<attribute name="POPULARITY" value="97" x="-20.32" y="-154.94" size="1.778" layer="27" display="off"/>
+<attribute name="VALUE" x="-18.415" y="-156.591" size="1.27" layer="27" ratio="10"/>
+</element>
+<element name="LED3" library="IDP_library" package="LED3MM" package3d_urn="urn:adsk.eagle:package:15797/1" value="LED_23MM" x="-20.32" y="-160.02" smashed="yes">
+<attribute name="NAME" x="-18.415" y="-159.639" size="1.27" layer="25" ratio="10"/>
+<attribute name="POPULARITY" value="97" x="-20.32" y="-160.02" size="1.778" layer="27" display="off"/>
+<attribute name="VALUE" x="-18.415" y="-161.671" size="1.27" layer="27" ratio="10"/>
+</element>
+<element name="LED4" library="IDP_library" package="LED3MM" package3d_urn="urn:adsk.eagle:package:15797/1" value="LED_23MM" x="-20.32" y="-165.1" smashed="yes">
+<attribute name="NAME" x="-18.415" y="-164.719" size="1.27" layer="25" ratio="10"/>
+<attribute name="POPULARITY" value="97" x="-20.32" y="-165.1" size="1.778" layer="27" display="off"/>
+<attribute name="VALUE" x="-18.415" y="-166.751" size="1.27" layer="27" ratio="10"/>
+</element>
+<element name="LED5" library="IDP_library" package="LED3MM" package3d_urn="urn:adsk.eagle:package:15797/1" value="LED_23MM" x="-20.32" y="-170.18" smashed="yes">
+<attribute name="NAME" x="-18.415" y="-169.799" size="1.27" layer="25" ratio="10"/>
+<attribute name="POPULARITY" value="97" x="-20.32" y="-170.18" size="1.778" layer="27" display="off"/>
+<attribute name="VALUE" x="-18.415" y="-171.831" size="1.27" layer="27" ratio="10"/>
+</element>
+<element name="U$2" library="IDP_library" package="TO92/" package3d_urn="urn:adsk.eagle:package:29930/3" value="HALL-SS495A" x="-27.94" y="-166.37" smashed="yes">
+<attribute name="NAME" x="-30.48" y="-163.322" size="1.27" layer="25" ratio="10"/>
+<attribute name="VALUE" x="-30.48" y="-170.688" size="1.27" layer="27" ratio="10"/>
+</element>
+<element name="IC1" library="IDP_library" package="DIL08" package3d_urn="urn:adsk.eagle:package:16409/2" value="LM311N" x="-22.86" y="-177.8" smashed="yes">
+<attribute name="NAME" x="-28.194" y="-180.721" size="1.27" layer="25" ratio="10" rot="R90"/>
+<attribute name="POPULARITY" value="4" x="-22.86" y="-177.8" size="1.778" layer="27" display="off"/>
+<attribute name="VALUE" x="-26.416" y="-178.435" size="1.27" layer="27" ratio="10"/>
 </element>
 </elements>
@@
 <contactref element="U$1" pad="P$1"/>
 <contactref element="J1" pad="4"/>
-<wire x1="-6.82" y1="-122.76" x2="-21.59" y2="-113.03" width="0" layer="19" extent="1-1"/>
+<contactref element="LED2" pad="K"/>
+<contactref element="LED5" pad="K"/>
+<contactref element="LED4" pad="K"/>
+<contactref element="LED3" pad="K"/>
+<contactref element="U$2" pad="2"/>
+<wire x1="-19.05" y1="-165.1" x2="-26.67" y2="-165.1" width="0" layer="19" extent="1-1"/>
+<wire x1="-19.05" y1="-170.18" x2="-19.05" y2="-165.1" width="0" layer="19" extent="1-1"/>
+<wire x1="-19.05" y1="-160.02" x2="-19.05" y2="-165.1" width="0" layer="19" extent="1-1"/>
+<wire x1="-19.05" y1="-154.94" x2="-19.05" y2="-160.02" width="0" layer="19" extent="1-1"/>
+<wire x1="-6.82" y1="-122.76" x2="-19.05" y2="-154.94" width="0" layer="19" extent="1-1"/>
 <wire x1="3.81" y1="-124.46" x2="-6.82" y2="-122.76" width="0" layer="19" extent="1-1"/>
+<wire x1="-21.59" y1="-113.03" x2="-6.82" y2="-122.76" width="0" layer="19" extent="1-1"/>
 <wire x1="2.54" y1="-105.41" x2="3.81" y2="-124.46" width="0" layer="19" extent="16-16"/>
 </signal>
@@
 <signal name="D0">
 <contactref element="M1" pad="D0"/>
+<contactref element="R6" pad="1"/>
+<wire x1="63.5" y1="-59.69" x2="-21.59" y2="-149.86" width="0" layer="19" extent="16-16"/>
 </signal>
 <signal name="D1">
 <contactref element="M1" pad="D1"/>
+<contactref element="R5" pad="1"/>
+<wire x1="60.96" y1="-59.69" x2="-21.59" y2="-143.51" width="0" layer="19" extent="16-16"/>
 </signal>
 <signal name="D2">
 <contactref element="M1" pad="D2"/>
+<contactref element="R4" pad="1"/>
+<wire x1="58.42" y1="-59.69" x2="-21.59" y2="-137.16" width="0" layer="19" extent="16-16"/>
 </signal>
 <signal name="D3">
 <contactref element="M1" pad="D3"/>
+<contactref element="R3" pad="1"/>
+<wire x1="55.88" y1="-59.69" x2="-21.59" y2="-130.81" width="0" layer="19" extent="16-16"/>
 </signal>
 <signal name="D4">
@@
 <contactref element="R2" pad="2"/>
 <contactref element="J1" pad="1"/>
+<contactref element="U$2" pad="3"/>
+<wire x1="-13.97" y1="-113.03" x2="-29.21" y2="-165.1" width="0" layer="19" extent="1-1"/>
 <wire x1="6.35" y1="-111.76" x2="-13.97" y2="-113.03" width="0" layer="19" extent="1-1"/>
 <wire x1="6.35" y1="-118.11" x2="6.35" y2="-111.76" width="0" layer="19" extent="1-1"/>
@@
 <wire x1="1.27" y1="-118.11" x2="1.27" y2="-124.46" width="0" layer="19" extent="1-1"/>
 </signal>
+<signal name="N$1">
+<contactref element="R3" pad="2"/>
+<contactref element="LED2" pad="A"/>
+<wire x1="-16.51" y1="-130.81" x2="-21.59" y2="-154.94" width="0" layer="19" extent="1-1"/>
+</signal>
+<signal name="N$2">
+<contactref element="R4" pad="2"/>
+<contactref element="LED3" pad="A"/>
+<wire x1="-16.51" y1="-137.16" x2="-21.59" y2="-160.02" width="0" layer="19" extent="1-1"/>
+</signal>
+<signal name="N$4">
+<contactref element="R5" pad="2"/>
+<contactref element="LED4" pad="A"/>
+<wire x1="-16.51" y1="-143.51" x2="-21.59" y2="-165.1" width="0" layer="19" extent="1-1"/>
+</signal>
+<signal name="N$5">
+<contactref element="R6" pad="2"/>
+<contactref element="LED5" pad="A"/>
+<wire x1="-16.51" y1="-149.86" x2="-21.59" y2="-170.18" width="0" layer="19" extent="1-1"/>
+</signal>
+<signal name="V+">
+<contactref element="IC1" pad="8"/>
+</signal>
+<signal name="V-">
+<contactref element="IC1" pad="4"/>
+</signal>
+<signal name="N$8">
+<contactref element="U$2" pad="1"/>
+<contactref element="IC1" pad="2"/>
+<wire x1="-26.67" y1="-167.64" x2="-24.13" y2="-181.61" width="0" layer="19" extent="1-1"/>
+</signal>
 </signals>
