File: Electronics/idp.brd (EAGLE design)
At the start: 100 x 80 mm, 16 parts, among them IC1 LM311N, J1 To IR Distance Sensor, M1 IDP_PROTOBOARD, T1 SFH 313 FA

Commit message: updated schematics
Parts:
- added J2: To Right IR Distance Sensor, IDP_library:7395-03
- J1: value To IR Distance Sensor -> To Left IR Distance Sensor
- R3: value R-EU_0207/5V -> 150k
Changed lines of the file:
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@@
 <attribute name="VALUE" x="5.7404" y="-126.2634" size="1.27" layer="27" ratio="10"/>
 </element>
-<element name="R3" library="IDP_library" package="0207/5V" package3d_urn="urn:adsk.eagle:package:23502/1" value="R-EU_0207/5V" x="-19.05" y="-130.81" smashed="yes">
+<element name="R3" library="IDP_library" package="0207/5V" package3d_urn="urn:adsk.eagle:package:23502/1" value="150k" x="-19.05" y="-130.81" smashed="yes">
 <attribute name="NAME" x="-20.193" y="-129.921" size="1.27" layer="25" ratio="10"/>
 <attribute name="POPULARITY" value="4" x="-19.05" y="-130.81" size="1.778" layer="27" display="off"/>
@@
 <attribute name="VALUE" x="-35.9156" y="-190.9826" size="0.9906" layer="27" ratio="10"/>
 </element>
-<element name="J1" library="IDP_library" package="7395-03" package3d_urn="urn:adsk.eagle:package:8078646/1" value="To IR Distance Sensor" x="-46.99" y="-177.8" smashed="yes">
+<element name="J1" library="IDP_library" package="7395-03" package3d_urn="urn:adsk.eagle:package:8078646/1" value="To Left IR Distance Sensor" x="-46.99" y="-177.8" smashed="yes">
 <attribute name="MF" value="MOLEX" x="-46.99" y="-177.8" size="1.778" layer="27" display="off"/>
 <attribute name="MPN" value="" x="-46.99" y="-177.8" size="1.778" layer="27" display="off"/>
@@
 <attribute name="VALUE" x="-42.3179" y="-180.2399" size="0.8128" layer="27" ratio="10" rot="R270"/>
 </element>
+<element name="J2" library="IDP_library" package="7395-03" package3d_urn="urn:adsk.eagle:package:8078646/1" value="To Right IR Distance Sensor" x="-57.15" y="-180.34" smashed="yes">
+<attribute name="MF" value="MOLEX" x="-57.15" y="-180.34" size="1.778" layer="27" display="off"/>
+<attribute name="MPN" value="" x="-57.15" y="-180.34" size="1.778" layer="27" display="off"/>
+<attribute name="NAME" x="-53.2399" y="-177.3921" size="1.016" layer="25" ratio="10" rot="R180"/>
+<attribute name="OC_FARNELL" value="unknown" x="-57.15" y="-180.34" size="1.778" layer="27" display="off"/>
+<attribute name="OC_NEWARK" value="unknown" x="-57.15" y="-180.34" size="1.778" layer="27" display="off"/>
+<attribute name="POPULARITY" value="0" x="-57.15" y="-180.34" size="1.778" layer="27" display="off"/>
+<attribute name="VALUE" x="-52.4779" y="-182.7799" size="0.8128" layer="27" ratio="10" rot="R270"/>
+</element>
 </elements>
