File: Electronics/idp.brd (EAGLE design)
At the start: 139.4 x 101.6 mm, 15 parts, among them J1 To Left IR Distance Sensor, J2 To Right IR Distance Sensor, M1 IDP_PROTOBOARD, T1 Phototransistor

Commit message: added LDR. created board
Parts:
- added LED6: Blue/Red, IDP_library:LED3MM
- added R7: 150, IDP_library:0204/7
- added R8: 10k, IDP_library:0204/7
- added U$1: LDR, IDP_library:LDR
- moved J2 67.5 mm to (34.3, 25.4), turned to 0 degrees
- moved J1 64.3 mm to (24.1, 25.4), turned to 0 degrees
- moved R2 58.6 mm to (39.4, 22.9)
- moved LED1 45.3 mm to (40.6, 26.7)
- moved LED4 45.0 mm to (62.2, 45.7), turned to 270 degrees
- moved R1 44.2 mm to (54.6, 20.3), turned to 180 degrees
- moved T1 39.9 mm to (54.6, 25.4)
- moved R6 32.1 mm to (57.1, 38.1), turned to 270 degrees
- moved LED5 30.5 mm to (57.1, 45.7), turned to 270 degrees
- moved R5 29.0 mm to (62.2, 38.1), turned to 270 degrees
- moved LED3 28.0 mm to (67.3, 45.7), turned to 270 degrees
- moved R3 27.9 mm to (72.4, 38.1), turned to 270 degrees
- moved LED2 22.5 mm to (72.4, 45.7), turned to 270 degrees
- moved R4 17.8 mm to (67.3, 38.1), turned to 270 degrees
Connections:
- new net A4: R8.1, U$1.P$2
- new net N$2: LED6.A, R7.1
- net +5V: now also R7.2, R8.2
- net GND: now also LED6.K, U$1.P$1
Routing:
- net +5V: track 0.00 -> 6.13 mm
- net N$5: track 0.00 -> 5.08 mm
- net N$4: track 0.00 -> 5.08 mm
- net N$12: track 0.00 -> 5.08 mm
- net N$1: track 0.00 -> 5.08 mm
- net N$2: track 0.00 -> 5.08 mm
- net A0: track 0.00 -> 5.08 mm
- net A4: track 0.00 -> 4.52 mm
- net N$3: track 0.00 -> 3.81 mm
