File: Electronics/idp.sch (EAGLE design)
At the start: 6 parts, among them J1 22-05-7048-04, M1 IDP_PROTOBOARD

Commit message: Updated eagle schematics
Parts:
- added IC1: LM311N, IDP_library:LM311N
- added LED2, LED3, LED4, LED5: LED_23MM, IDP_library:LED_23MM
- added R3, R4, R5, R6: R-EU_0207/5V, IDP_library:R-EU_0207/5V
- added U$2: HALL-SS495A, IDP_library:HALL-SS495A
Connections:
- new net N$1: LED2.A, R3.2
- new net N$2: LED3.A, R4.2
- new net N$4: LED4.A, R5.2
- new net N$5: LED5.A, R6.2
- new net N$8: IC1.+IN, U$2.V+
- net +5V: now also U$2.VS
- net D0: now also R6.1
- net D1: now also R5.1
- net D2: now also R4.1
- net D3: now also R3.1
- net GND: now also LED2.C, LED3.C, LED4.C, LED5.C, U$2.V-
Changed lines of the file:
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@@
 <part name="P+3" library="IDP_library" deviceset="+5V" device=""/>
 <part name="GND3" library="IDP_library" deviceset="GND" device=""/>
+<part name="R3" library="IDP_library" deviceset="R-EU_" device="0207/5V" package3d_urn="urn:adsk.eagle:package:23502/1"/>
+<part name="R4" library="IDP_library" deviceset="R-EU_" device="0207/5V" package3d_urn="urn:adsk.eagle:package:23502/1"/>
+<part name="R5" library="IDP_library" deviceset="R-EU_" device="0207/5V" package3d_urn="urn:adsk.eagle:package:23502/1"/>
+<part name="R6" library="IDP_library" deviceset="R-EU_" device="0207/5V" package3d_urn="urn:adsk.eagle:package:23502/1"/>
+<part name="LED2" library="IDP_library" deviceset="LED_2" device="3MM" package3d_urn="urn:adsk.eagle:package:15797/1"/>
+<part name="LED3" library="IDP_library" deviceset="LED_2" device="3MM" package3d_urn="urn:adsk.eagle:package:15797/1"/>
+<part name="LED4" library="IDP_library" deviceset="LED_2" device="3MM" package3d_urn="urn:adsk.eagle:package:15797/1"/>
+<part name="LED5" library="IDP_library" deviceset="LED_2" device="3MM" package3d_urn="urn:adsk.eagle:package:15797/1"/>
+<part name="GND4" library="IDP_library" deviceset="GND" device=""/>
+<part name="U$2" library="IDP_library" deviceset="HALL-SS495A" device="" package3d_urn="urn:adsk.eagle:package:29930/3"/>
+<part name="IC1" library="IDP_library" deviceset="LM311" device="N" package3d_urn="urn:adsk.eagle:package:16409/2"/>
+<part name="P+4" library="IDP_library" deviceset="+5V" device=""/>
+<part name="GND5" library="IDP_library" deviceset="GND" device=""/>
 </parts>
 <sheets>
@@
 <attribute name="VALUE" x="177.8" y="121.92" size="1.778" layer="96"/>
 </instance>
+<instance part="R3" gate="G$1" x="170.18" y="106.68" smashed="yes">
+<attribute name="NAME" x="168.91" y="105.6386" size="1.778" layer="95"/>
+</instance>
+<instance part="R4" gate="G$1" x="170.18" y="104.14" smashed="yes">
+<attribute name="NAME" x="168.91" y="103.0986" size="1.778" layer="95"/>
+</instance>
+<instance part="R5" gate="G$1" x="170.18" y="101.6" smashed="yes">
+<attribute name="NAME" x="168.91" y="100.5586" size="1.778" layer="95"/>
+</instance>
+<instance part="R6" gate="G$1" x="170.18" y="99.06" smashed="yes">
+<attribute name="NAME" x="168.91" y="98.0186" size="1.778" layer="95"/>
+</instance>
+<instance part="LED2" gate="G$1" x="182.88" y="106.68" smashed="yes" rot="R90"/>
+<instance part="LED3" gate="G$1" x="182.88" y="104.14" smashed="yes" rot="R90">
+<attribute name="NAME" x="187.452" y="105.156" size="1.778" layer="95" rot="R180"/>
+</instance>
+<instance part="LED4" gate="G$1" x="182.88" y="101.6" smashed="yes" rot="R90">
+<attribute name="NAME" x="187.452" y="102.616" size="1.778" layer="95" rot="R180"/>
+</instance>
+<instance part="LED5" gate="G$1" x="182.88" y="99.06" smashed="yes" rot="R90">
+<attribute name="NAME" x="187.452" y="100.076" size="1.778" layer="95" rot="R180"/>
+</instance>
+<instance part="GND4" gate="1" x="193.04" y="93.98" smashed="yes">
+<attribute name="VALUE" x="190.5" y="91.44" size="1.778" layer="96"/>
+</instance>
+<instance part="U$2" gate="G$1" x="124.46" y="71.12" smashed="yes"/>
+<instance part="IC1" gate="A" x="144.78" y="60.96" smashed="yes">
+<attribute name="NAME" x="147.32" y="66.675" size="1.778" layer="95"/>
+<attribute name="VALUE" x="147.32" y="55.88" size="1.778" layer="96"/>
+</instance>
+<instance part="P+4" gate="1" x="121.92" y="66.04" smashed="yes" rot="R90">
+<attribute name="VALUE" x="127" y="63.5" size="1.778" layer="96" rot="R180"/>
+</instance>
+<instance part="GND5" gate="1" x="129.54" y="60.96" smashed="yes">
+<attribute name="VALUE" x="127" y="58.42" size="1.778" layer="96"/>
+</instance>
 </instances>
 <busses>
@@
 <segment>
 <pinref part="M1" gate="G$1" pin="D0"/>
-<wire x1="144.78" y1="99.06" x2="162.56" y2="99.06" width="0.1524" layer="91"/>
+<wire x1="144.78" y1="99.06" x2="165.1" y2="99.06" width="0.1524" layer="91"/>
 <label x="160.02" y="99.06" size="1.778" layer="95" align="bottom-right"/>
+<pinref part="R6" gate="G$1" pin="1"/>
 </segment>
 </net>
@@
 <segment>
 <pinref part="M1" gate="G$1" pin="D1"/>
-<wire x1="144.78" y1="101.6" x2="162.56" y2="101.6" width="0.1524" layer="91"/>
+<wire x1="144.78" y1="101.6" x2="165.1" y2="101.6" width="0.1524" layer="91"/>
 <label x="160.02" y="101.6" size="1.778" layer="95" align="bottom-right"/>
+<pinref part="R5" gate="G$1" pin="1"/>
 </segment>
 </net>
@@
 <segment>
 <pinref part="M1" gate="G$1" pin="D2"/>
-<wire x1="144.78" y1="104.14" x2="162.56" y2="104.14" width="0.1524" layer="91"/>
+<wire x1="144.78" y1="104.14" x2="165.1" y2="104.14" width="0.1524" layer="91"/>
 <label x="160.02" y="104.14" size="1.778" layer="95" align="bottom-right"/>
+<pinref part="R4" gate="G$1" pin="1"/>
 </segment>
 </net>
@@
 <segment>
 <pinref part="M1" gate="G$1" pin="D3"/>
-<wire x1="144.78" y1="106.68" x2="162.56" y2="106.68" width="0.1524" layer="91"/>
+<wire x1="144.78" y1="106.68" x2="165.1" y2="106.68" width="0.1524" layer="91"/>
 <label x="160.02" y="106.68" size="1.778" layer="95" align="bottom-right"/>
+<pinref part="R3" gate="G$1" pin="1"/>
 </segment>
 </net>
@@
 <wire x1="180.34" y1="129.54" x2="185.42" y2="129.54" width="0.1524" layer="91"/>
 </segment>
+<segment>
+<pinref part="LED2" gate="G$1" pin="C"/>
+<wire x1="187.96" y1="106.68" x2="193.04" y2="106.68" width="0.1524" layer="91"/>
+<pinref part="GND4" gate="1" pin="GND"/>
+<wire x1="193.04" y1="106.68" x2="193.04" y2="104.14" width="0.1524" layer="91"/>
+<pinref part="LED5" gate="G$1" pin="C"/>
+<wire x1="193.04" y1="104.14" x2="193.04" y2="101.6" width="0.1524" layer="91"/>
+<wire x1="193.04" y1="101.6" x2="193.04" y2="99.06" width="0.1524" layer="91"/>
+<wire x1="193.04" y1="99.06" x2="193.04" y2="96.52" width="0.1524" layer="91"/>
+<wire x1="187.96" y1="99.06" x2="193.04" y2="99.06" width="0.1524" layer="91"/>
+<junction x="193.04" y="99.06"/>
+<pinref part="LED4" gate="G$1" pin="C"/>
+<wire x1="187.96" y1="101.6" x2="193.04" y2="101.6" width="0.1524" layer="91"/>
+<junction x="193.04" y="101.6"/>
+<pinref part="LED3" gate="G$1" pin="C"/>
+<wire x1="187.96" y1="104.14" x2="193.04" y2="104.14" width="0.1524" layer="91"/>
+<junction x="193.04" y="104.14"/>
+</segment>
+<segment>
+<pinref part="U$2" gate="G$1" pin="V-"/>
+<wire x1="129.54" y1="66.04" x2="129.54" y2="63.5" width="0.1524" layer="91"/>
+<pinref part="GND5" gate="1" pin="GND"/>
+</segment>
 </net>
 <net name="AREF" class="0">
@@
 <pinref part="P+3" gate="1" pin="+5V"/>
 </segment>
+<segment>
+<pinref part="U$2" gate="G$1" pin="VS"/>
+<wire x1="127" y1="66.04" x2="124.46" y2="66.04" width="0.1524" layer="91"/>
+<pinref part="P+4" gate="1" pin="+5V"/>
+</segment>
 </net>
 <net name="N$3" class="0">
@@
 </segment>
 </net>
+<net name="N$1" class="0">
+<segment>
+<pinref part="R3" gate="G$1" pin="2"/>
+<pinref part="LED2" gate="G$1" pin="A"/>
+<wire x1="175.26" y1="106.68" x2="180.34" y2="106.68" width="0.1524" layer="91"/>
+</segment>
+</net>
+<net name="N$2" class="0">
+<segment>
+<pinref part="R4" gate="G$1" pin="2"/>
+<pinref part="LED3" gate="G$1" pin="A"/>
+<wire x1="175.26" y1="104.14" x2="180.34" y2="104.14" width="0.1524" layer="91"/>
+</segment>
+</net>
+<net name="N$4" class="0">
+<segment>
+<pinref part="R5" gate="G$1" pin="2"/>
+<pinref part="LED4" gate="G$1" pin="A"/>
+<wire x1="175.26" y1="101.6" x2="180.34" y2="101.6" width="0.1524" layer="91"/>
+</segment>
+</net>
+<net name="N$5" class="0">
+<segment>
+<pinref part="R6" gate="G$1" pin="2"/>
+<pinref part="LED5" gate="G$1" pin="A"/>
+<wire x1="175.26" y1="99.06" x2="180.34" y2="99.06" width="0.1524" layer="91"/>
+</segment>
+</net>
+<net name="N$8" class="0">
+<segment>
+<pinref part="U$2" gate="G$1" pin="V+"/>
+<wire x1="132.08" y1="66.04" x2="132.08" y2="63.5" width="0.1524" layer="91"/>
+<pinref part="IC1" gate="A" pin="+IN"/>
+<wire x1="132.08" y1="63.5" x2="137.16" y2="63.5" width="0.1524" layer="91"/>
+</segment>
+</net>
