File: Electronics/idp.sch (EAGLE design)
At the start: 16 parts, among them IC1 LM311N, J1 To IR Distance Sensor, M1 IDP_PROTOBOARD, T1 SFH 313 FA

Commit message: updated schematics
Parts:
- added J2: To Right IR Distance Sensor, IDP_library:22-05-7038-03
- J1: value To IR Distance Sensor -> To Left IR Distance Sensor
- R3: value R-EU_0207/5V -> 150k
Other:
- moved on the sheet: LED3, LED4, LED5
Changed lines of the file:
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@@
 <part name="GND1" library="IDP_library" deviceset="GND" device=""/>
 <part name="GND2" library="IDP_library" deviceset="GND" device=""/>
-<part name="R3" library="IDP_library" deviceset="R-EU_" device="0207/5V" package3d_urn="urn:adsk.eagle:package:23502/1"/>
+<part name="R3" library="IDP_library" deviceset="R-EU_" device="0207/5V" package3d_urn="urn:adsk.eagle:package:23502/1" value="150k"/>
 <part name="R4" library="IDP_library" deviceset="R-EU_" device="0207/5V" package3d_urn="urn:adsk.eagle:package:23502/1"/>
 <part name="R5" library="IDP_library" deviceset="R-EU_" device="0207/5V" package3d_urn="urn:adsk.eagle:package:23502/1"/>
@@
 <part name="R2" library="IDP_library" deviceset="R-EU_" device="0204/7" package3d_urn="urn:adsk.eagle:package:23498/2" value="150"/>
 <part name="R1" library="IDP_library" deviceset="R-EU_" device="0204/7" package3d_urn="urn:adsk.eagle:package:23498/2" value="10k"/>
-<part name="J1" library="IDP_library" deviceset="22-?-03" device="05-7038" package3d_urn="urn:adsk.eagle:package:8078646/1" value="To IR Distance Sensor"/>
+<part name="J1" library="IDP_library" deviceset="22-?-03" device="05-7038" package3d_urn="urn:adsk.eagle:package:8078646/1" value="To Left IR Distance Sensor"/>
 <part name="P+3" library="IDP_library" deviceset="+5V" device=""/>
 <part name="GND3" library="IDP_library" deviceset="GND" device=""/>
+<part name="J2" library="IDP_library" deviceset="22-?-03" device="05-7038" package3d_urn="urn:adsk.eagle:package:8078646/1" value="To Right IR Distance Sensor"/>
 </parts>
 <sheets>
@@
 <attribute name="NAME" x="168.91" y="98.0186" size="1.778" layer="95"/>
 </instance>
-<instance part="LED2" gate="G$1" x="182.88" y="106.68" smashed="yes" rot="R90"/>
-<instance part="LED3" gate="G$1" x="182.88" y="104.14" smashed="yes" rot="R90">
-<attribute name="NAME" x="187.452" y="105.156" size="1.778" layer="95" rot="R180"/>
-</instance>
-<instance part="LED4" gate="G$1" x="182.88" y="101.6" smashed="yes" rot="R90">
-<attribute name="NAME" x="187.452" y="102.616" size="1.778" layer="95" rot="R180"/>
-</instance>
-<instance part="LED5" gate="G$1" x="182.88" y="99.06" smashed="yes" rot="R90">
-<attribute name="NAME" x="187.452" y="100.076" size="1.778" layer="95" rot="R180"/>
+<instance part="LED2" gate="G$1" x="190.5" y="106.68" smashed="yes" rot="R90"/>
+<instance part="LED3" gate="G$1" x="185.42" y="104.14" smashed="yes" rot="R90">
+<attribute name="NAME" x="189.992" y="115.316" size="1.778" layer="95" rot="R180"/>
+</instance>
+<instance part="LED4" gate="G$1" x="180.34" y="101.6" smashed="yes" rot="R90">
+<attribute name="NAME" x="179.832" y="102.616" size="1.778" layer="95" rot="R180"/>
+</instance>
+<instance part="LED5" gate="G$1" x="175.26" y="99.06" smashed="yes" rot="R90">
+<attribute name="NAME" x="174.752" y="97.536" size="1.778" layer="95" rot="R180"/>
 </instance>
 <instance part="GND4" gate="1" x="193.04" y="93.98" smashed="yes">
@@
 <instance part="T1" gate="G$1" x="73.66" y="55.88" smashed="yes">
 <attribute name="NAME" x="66.04" y="53.34" size="1.778" layer="95" rot="R90"/>
-<attribute name="VALUE" x="60.96" y="60.96" size="1.778" layer="96" rot="R270"/>
 </instance>
 <instance part="R2" gate="G$1" x="88.9" y="71.12" smashed="yes" rot="R90">
@@
 <instance part="GND3" gate="1" x="55.88" y="88.9" smashed="yes">
 <attribute name="VALUE" x="53.34" y="86.36" size="1.778" layer="96"/>
+</instance>
+<instance part="J2" gate="G$1" x="40.64" y="76.2" smashed="yes">
+<attribute name="VALUE" x="36.83" y="66.04" size="1.778" layer="96" rot="R90"/>
+<attribute name="NAME" x="34.29" y="74.422" size="1.778" layer="95" rot="R90"/>
 </instance>
 </instances>
@@
 <segment>
 <pinref part="LED2" gate="G$1" pin="C"/>
-<wire x1="187.96" y1="106.68" x2="193.04" y2="106.68" width="0.1524" layer="91"/>
+<wire x1="195.58" y1="106.68" x2="193.04" y2="106.68" width="0.1524" layer="91"/>
 <pinref part="GND4" gate="1" pin="GND"/>
 <wire x1="193.04" y1="106.68" x2="193.04" y2="104.14" width="0.1524" layer="91"/>
@@
 <wire x1="193.04" y1="101.6" x2="193.04" y2="99.06" width="0.1524" layer="91"/>
 <wire x1="193.04" y1="99.06" x2="193.04" y2="96.52" width="0.1524" layer="91"/>
-<wire x1="187.96" y1="99.06" x2="193.04" y2="99.06" width="0.1524" layer="91"/>
+<wire x1="180.34" y1="99.06" x2="193.04" y2="99.06" width="0.1524" layer="91"/>
 <junction x="193.04" y="99.06"/>
 <pinref part="LED4" gate="G$1" pin="C"/>
-<wire x1="187.96" y1="101.6" x2="193.04" y2="101.6" width="0.1524" layer="91"/>
+<wire x1="185.42" y1="101.6" x2="193.04" y2="101.6" width="0.1524" layer="91"/>
 <junction x="193.04" y="101.6"/>
 <pinref part="LED3" gate="G$1" pin="C"/>
-<wire x1="187.96" y1="104.14" x2="193.04" y2="104.14" width="0.1524" layer="91"/>
+<wire x1="190.5" y1="104.14" x2="193.04" y2="104.14" width="0.1524" layer="91"/>
 <junction x="193.04" y="104.14"/>
 </segment>
@@
 <pinref part="R3" gate="G$1" pin="2"/>
 <pinref part="LED2" gate="G$1" pin="A"/>
-<wire x1="175.26" y1="106.68" x2="180.34" y2="106.68" width="0.1524" layer="91"/>
+<wire x1="175.26" y1="106.68" x2="187.96" y2="106.68" width="0.1524" layer="91"/>
 </segment>
 </net>
@@
 <pinref part="R4" gate="G$1" pin="2"/>
 <pinref part="LED3" gate="G$1" pin="A"/>
-<wire x1="175.26" y1="104.14" x2="180.34" y2="104.14" width="0.1524" layer="91"/>
+<wire x1="182.88" y1="104.14" x2="175.26" y2="104.14" width="0.1524" layer="91"/>
 </segment>
 </net>
@@
 <pinref part="R5" gate="G$1" pin="2"/>
 <pinref part="LED4" gate="G$1" pin="A"/>
-<wire x1="175.26" y1="101.6" x2="180.34" y2="101.6" width="0.1524" layer="91"/>
+<wire x1="175.26" y1="101.6" x2="177.8" y2="101.6" width="0.1524" layer="91"/>
 </segment>
 </net>
@@
 <pinref part="R6" gate="G$1" pin="2"/>
 <pinref part="LED5" gate="G$1" pin="A"/>
-<wire x1="175.26" y1="99.06" x2="180.34" y2="99.06" width="0.1524" layer="91"/>
-</segment>
-</net>
+<wire x1="172.72" y1="99.06" x2="175.26" y2="99.06" width="0.1524" layer="91"/>
+</segment>
+</net>
